File: v2/kicad/flutter_v2_wren.kicad_pcb (KiCad board)
At the start: 2 copper layers, 173.5 x 108.6 mm, 88 parts

Commit message: update
Parts:
- added G***: LOGO, LOGO, F.Cu at (80.1, 8.62)
- added G***: LOGO, LOGO, F.Cu at (125.1, 13.4)
- added REF**: MountingHole_2.2mm_M2_DIN965_Pad, MountingHole:MountingHole_2.2mm_M2_DIN965_Pad, F.Cu at (-9.32, 6.07)
- added REF**: MountingHole_2.2mm_M2_DIN965_Pad, MountingHole:MountingHole_2.2mm_M2_DIN965_Pad, F.Cu at (138.1, 3.22)
- added REF**: MountingHole_2.2mm_M2_DIN965_Pad, MountingHole:MountingHole_2.2mm_M2_DIN965_Pad, F.Cu at (149.0, 57.1)
- added REF**: MountingHole_2.2mm_M2_DIN965_Pad, MountingHole:MountingHole_2.2mm_M2_DIN965_Pad, F.Cu at (-9.32, -41.4)
- added REF**: MountingHole_2.2mm_M2_DIN965_Pad, MountingHole:MountingHole_2.2mm_M2_DIN965_Pad, F.Cu at (161.2, 38.3)
- added REF**: MountingHole_2.2mm_M2_DIN965_Pad, MountingHole:MountingHole_2.2mm_M2_DIN965_Pad, F.Cu at (61.7, 9.57)
- added REF**: MountingHole_2.2mm_M2_DIN965_Pad, MountingHole:MountingHole_2.2mm_M2_DIN965_Pad, F.Cu at (99.7, -45.5)
- moved ? 1.48 mm to (120.7, -12.4)
Routing:
- net pos: track 28.1 -> 29.7 mm
- net GND: track 83.4 -> 85.0 mm
- net P0: track 269.8 -> 270.5 mm
Other:
- board size 173.5 x 108.6 mm -> 175.9 x 108.6 mm
- board text added: "+"
- board text added: "ON"
- board text added: "Sep. 2022"
- board text added: "V2 By Trent Slutzky"
- board text added: "flash"
